File: pcb/pcb.kicad_pcb (KiCad board)
At the start: 2 copper layers, 0 parts

Commit message: PCB mid-way
Parts:
- added C1: 100n, Capacitor_SMD:C_1206_3216Metric_Pad1.33x1.80mm_HandSolder, F.Cu at (87.5, 80.5)
- added C10: 33p, Capacitor_SMD:C_1206_3216Metric_Pad1.33x1.80mm_HandSolder, F.Cu at (76.9, 97.5)
- added C11: 100n, Capacitor_SMD:C_1206_3216Metric_Pad1.33x1.80mm_HandSolder, F.Cu at (153.5, 75.4)
- added C12: 10u, Capacitor_SMD:C_1206_3216Metric_Pad1.33x1.80mm_HandSolder, F.Cu at (94.0, 67.9)
- added C13: 100n, Capacitor_SMD:C_1206_3216Metric_Pad1.33x1.80mm_HandSolder, F.Cu at (98.5, 67.9)
- added C2: 10u, Capacitor_SMD:C_1206_3216Metric_Pad1.33x1.80mm_HandSolder, F.Cu at (87.4, 76.5)
- added C3: 100n, Capacitor_SMD:C_1206_3216Metric_Pad1.33x1.80mm_HandSolder, F.Cu at (98.0, 86.4)
- added C4: 100n, Capacitor_SMD:C_1206_3216Metric_Pad1.33x1.80mm_HandSolder, F.Cu at (92.9, 96.5)
- added C5: 100n, Capacitor_SMD:C_1206_3216Metric_Pad1.33x1.80mm_HandSolder, F.Cu at (82.0, 89.8)
- added C6: 100n, Capacitor_SMD:C_1206_3216Metric_Pad1.33x1.80mm_HandSolder, F.Cu at (82.0, 83.9)
- added C7: 100n, Capacitor_SMD:C_1206_3216Metric_Pad1.33x1.80mm_HandSolder, F.Cu at (80.0, 67.0)
- added C8: 10u, Capacitor_SMD:C_1206_3216Metric_Pad1.33x1.80mm_HandSolder, F.Cu at (76.0, 66.9)
- added C9: 33p, Capacitor_SMD:C_1206_3216Metric_Pad1.33x1.80mm_HandSolder, F.Cu at (76.3, 79.0)
- added D1: LED, LED_SMD:LED_1206_3216Metric_Pad1.42x1.75mm_HandSolder, F.Cu at (100.0, 76.5)
- added D2: LED, LED_SMD:LED_1206_3216Metric_Pad1.42x1.75mm_HandSolder, F.Cu at (141.5, 95.5)
- added D3: LED, LED_SMD:LED_1206_3216Metric_Pad1.42x1.75mm_HandSolder, F.Cu at (141.5, 98.9)
- added D4: LED, LED_SMD:LED_1206_3216Metric_Pad1.42x1.75mm_HandSolder, F.Cu at (141.5, 102.3)
- added D5: LED, LED_SMD:LED_1206_3216Metric_Pad1.42x1.75mm_HandSolder, F.Cu at (141.5, 105.7)
- added D6: LED, LED_SMD:LED_1206_3216Metric_Pad1.42x1.75mm_HandSolder, F.Cu at (141.5, 109.1)
- added D7: LED, LED_SMD:LED_1206_3216Metric_Pad1.42x1.75mm_HandSolder, F.Cu at (141.5, 112.5)
- added D8: LED, LED_SMD:LED_1206_3216Metric_Pad1.42x1.75mm_HandSolder, F.Cu at (141.5, 115.9)
- added D9: LED, LED_SMD:LED_1206_3216Metric_Pad1.42x1.75mm_HandSolder, F.Cu at (141.5, 119.3)
- added J1: GPIO, Connector_PinHeader_2.54mm:PinHeader_1x03_P2.54mm_Vertical, F.Cu at (176.7, 76.0)
- added J2: 3.3V Power, Connector_PinHeader_2.54mm:PinHeader_1x02_P2.54mm_Vertical, F.Cu at (156.6, 92.8)
- added J3: 3.3V Power, Connector_PinHeader_2.54mm:PinHeader_1x02_P2.54mm_Vertical, F.Cu at (161.2, 92.8)
- added J4: SPI2, Connector_PinHeader_2.54mm:PinHeader_1x06_P2.54mm_Vertical, F.Cu at (146.8, 106.6)
- added J5: SWD, Connector_PinHeader_2.54mm:PinHeader_1x05_P2.54mm_Vertical, F.Cu at (81.4, 58.5)
- added J6: 5V Power, Connector_PinHeader_2.54mm:PinHeader_1x02_P2.54mm_Vertical, F.Cu at (165.8, 92.8)
- added J7: 5V Power, Connector_PinHeader_2.54mm:PinHeader_1x02_P2.54mm_Vertical, F.Cu at (170.4, 92.8)
- added J8: I2C2, Connector_PinHeader_2.54mm:PinHeader_1x04_P2.54mm_Vertical, F.Cu at (156.6, 111.2)
- added J9: USART1, Connector_PinHeader_2.54mm:PinHeader_1x04_P2.54mm_Vertical, F.Cu at (161.2, 111.2)
- added R1: 10k, Resistor_SMD:R_1206_3216Metric_Pad1.30x1.75mm_HandSolder, F.Cu at (159.5, 75.4)
- added R10: 1.5K, Resistor_SMD:R_1206_3216Metric_Pad1.30x1.75mm_HandSolder, F.Cu at (171.4, 78.7)
- added R11: 1.5K, Resistor_SMD:R_1206_3216Metric_Pad1.30x1.75mm_HandSolder, F.Cu at (171.4, 82.0)
- added R12: 1.5K, Resistor_SMD:R_1206_3216Metric_Pad1.30x1.75mm_HandSolder, F.Cu at (171.4, 85.3)
- added R2: 1.5K, Resistor_SMD:R_1206_3216Metric_Pad1.30x1.75mm_HandSolder, F.Cu at (94.0, 76.5)
- added R3: R, Resistor_SMD:R_1206_3216Metric_Pad1.30x1.75mm_HandSolder, F.Cu at (159.5, 82.0)
- added R4: R, Resistor_SMD:R_1206_3216Metric_Pad1.30x1.75mm_HandSolder, F.Cu at (159.5, 85.3)
- added R5: 1.5K, Resistor_SMD:R_1206_3216Metric_Pad1.30x1.75mm_HandSolder, F.Cu at (165.5, 75.4)
- added R6: 1.5K, Resistor_SMD:R_1206_3216Metric_Pad1.30x1.75mm_HandSolder, F.Cu at (165.5, 78.7)
- added R7: 1.5K, Resistor_SMD:R_1206_3216Metric_Pad1.30x1.75mm_HandSolder, F.Cu at (165.5, 82.0)
- added R8: 1.5K, Resistor_SMD:R_1206_3216Metric_Pad1.30x1.75mm_HandSolder, F.Cu at (165.5, 85.3)
- added R9: 1.5K, Resistor_SMD:R_1206_3216Metric_Pad1.30x1.75mm_HandSolder, F.Cu at (171.4, 75.4)
- added SW1: SW_Push, Button_Switch_SMD:SW_SPST_PTS647_Sx38, F.Cu at (169.9, 115.9)
- added SW2: SW_SPDT, Button_Switch_SMD:SW_SPDT_PCM12, F.Cu at (149.4, 93.4)
- added SW3: SW_SPDT, Button_Switch_SMD:SW_SPDT_PCM12, F.Cu at (149.4, 100.3)
- added U1: STM32F103C8T6, Package_QFP:LQFP-48_7x7mm_P0.5mm, F.Cu at (90.2, 88.6)
- added U2: AMS1117-3.3, Package_TO_SOT_SMD:SOT-223-3_TabPin2, F.Cu at (86.5, 68.0)
- added Y1: 8MHz, Crystal:Crystal_SMD_HC49-SD, F.Cu at (74.9, 88.2)

Commit message: PCB Setting done
Parts:
- moved SW1 102.1 mm to (76.6, 74.5)
- moved J1 96.4 mm to (83.0, 98.3), turned to 90 degrees
- moved R5 92.9 mm to (77.2, 104.0), turned to 90 degrees
- moved R6 88.0 mm to (81.2, 104.0), turned to 90 degrees
- moved SW3 84.2 mm to (72.3, 66.6), turned to -90 degrees
- moved R9 83.3 mm to (93.2, 104.0), turned to 90 degrees
- moved R7 83.2 mm to (85.2, 104.0), turned to 90 degrees
- moved R8 78.4 mm to (89.3, 104.0), turned to 90 degrees
- moved R10 78.4 mm to (97.2, 104.0), turned to 90 degrees
- moved J7 76.5 mm to (100.2, 62.5), turned to 90 degrees
- moved J6 74.2 mm to (100.0, 58.5), turned to 90 degrees
- moved R11 73.9 mm to (100.8, 104.0), turned to 90 degrees
- moved C11 71.4 mm to (82.2, 77.7), turned to -90 degrees
- moved R12 69.0 mm to (105.0, 104.0), turned to 90 degrees
- moved D2 66.1 mm to (77.2, 110.3), turned to -90 degrees
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
Commit message: PCB almost done, proctored by Parul
Parts:
- moved J9 17.3 mm to (100.7, 81.0)
- moved J5 12.8 mm to (94.1, 60.0), turned to -90 degrees
- moved J4 12.2 mm to (97.5, 93.3)
- moved R12 7.80 mm to (109.5, 110.4), turned to -90 degrees
- moved R11 7.33 mm to (104.5, 110.4), turned to -90 degrees
- moved D9 7.27 mm to (109.5, 104.8), turned to 90 degrees
- moved R5 6.92 mm to (74.4, 110.4), turned to -90 degrees
- moved R10 6.75 mm to (99.5, 110.4), turned to -90 degrees
- moved D8 6.65 mm to (104.5, 104.8), turned to 90 degrees
- moved R6 6.61 mm to (79.4, 110.4), turned to -90 degrees
- moved R9 6.48 mm to (94.5, 110.4), turned to -90 degrees
- moved R7 6.40 mm to (84.4, 110.4), turned to -90 degrees
- moved R8 6.35 mm to (89.5, 110.4), turned to -90 degrees
- moved D2 6.16 mm to (74.4, 104.8), turned to 90 degrees
- moved D7 6.03 mm to (99.5, 104.8), turned to 90 degrees
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Connections:
- J4 pad 2: /MISO -> /CS
- J4 pad 3: /MOSI -> /CLK
- J4 pad 4: /CLK -> /MISO
- J4 pad 5: /CS -> /MOSI
Routing:
- net /5V_IN: track 0.00 -> 33.2 mm
- net /SCL: track 0.00 -> 30.4 mm, vias 0 -> 1
- net /LED7: track 0.00 -> 27.4 mm
- net /SWDCLK: track 0.00 -> 27.2 mm, vias 0 -> 1
- net /SDA: track 0.00 -> 26.9 mm, vias 0 -> 1
- net /SWDIO: track 0.00 -> 26.4 mm, vias 0 -> 1
- net +3.3V: track 0.00 -> 23.9 mm
- net /LED6: track 0.00 -> 22.8 mm
- net GND: track 0.00 -> 21.0 mm
- net /LED0: track 0.00 -> 20.1 mm
- net /RX: track 0.00 -> 19.4 mm
- net /LED5: track 0.00 -> 18.4 mm
- net /TX: track 0.00 -> 18.1 mm
- net /HSE_IN: track 0.00 -> 17.4 mm
- net /LED1: track 0.00 -> 16.9 mm
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Other:
- board outline added: 40.7 x 58.1 mm

Commit message: Completed routing with some silkscreen
Parts:
- moved D1 5.80 mm to (94.5, 74.8), turned to -90 degrees
- moved R2 4.56 mm to (98.2, 74.8), turned to 90 degrees
- moved J9 1.53 mm to (100.7, 79.5)
- moved C7 1.35 mm to (83.2, 66.5)
- moved C8 1.35 mm to (79.5, 66.6)
- moved J3 0.81 mm to (107.7, 61.8)
- moved J6 0.81 mm to (100.4, 57.7)
- moved J7 0.81 mm to (100.6, 61.7)
- moved J2 0.81 mm to (107.7, 57.8)
- moved SW1 0.65 mm to (77.2, 74.5)
- moved SW2 0.64 mm to (109.7, 71.2)
- moved C4 0.63 mm to (94.8, 96.5)
- turned C13 to -90 degrees
Connections:
- J8 pad 2: /SCL -> /SDA
- J8 pad 3: /SDA -> /SCL
- R3 pad 2: /SCL -> /SDA
- R4 pad 2: /SDA -> /SCL
Routing:
- net GND: track 21.0 -> 144.0 mm, vias 0 -> 5
- net +3.3V: track 23.9 -> 70.9 mm, vias 0 -> 8
- net Net-(SW3-A): track 0.00 -> 35.2 mm
- net /3.3V_IN: track 0.00 -> 30.6 mm
- net /BOOT: track 0.00 -> 22.6 mm, vias 0 -> 2
- net /NRST: track 5.73 -> 22.6 mm
- net /LED4: track 7.59 -> 14.0 mm
- net /5V_IN: track 33.2 -> 26.9 mm
- net Net-(SW2-B): track 0.00 -> 4.54 mm
- net Net-(D1-A): track 0.00 -> 3.77 mm
- net /RX: track 19.4 -> 16.6 mm
- net /SCL: track 30.4 -> 32.5 mm
- net /CS: track 8.51 -> 6.50 mm
- net /SDA: track 26.9 -> 28.8 mm
- net /TX: track 18.1 -> 19.2 mm
- added copper zone on F.Cu, net +3.3V
- added copper zone on B.Cu, net GND
Other:
- board size 40.7 x 58.1 mm -> 40.7 x 59.1 mm
- board text added: "3.3V"
- board text added: "5V"
- board text added: "CLK"
- board text added: "CS"
- board text added: "GND"
- board text added: "MISO"
- board text added: "MOSI"
- board text added: "NRST"
- board text added: "PC13"
- board text added: "PC14"
- board text added: "PC15"
- board text added: "RX"
- board text added: "SCL"
- board text added: "SDA"
- board text added: "SWCK"
- board text added: "SWIO"
- board text added: "TX"

Commit message: Finished PCB
Parts:
- added G***: LOGO, LOGO, B.Cu at (90.8, 84.0)
- moved C3 2.63 mm to (99.0, 84.0), turned to 180 degrees
- moved R3 0.85 mm to (103.4, 85.0)
- moved R4 0.85 mm to (107.5, 85.0)
- moved R1 0.80 mm to (104.5, 72.0)
Connections:
- U1 pad 34: unconnected-(U1-PA13-Pad34) -> /SWDIO
- U1 pad 37: /SWDIO -> /SWDCLK
- U1 pad 38: /SWDCLK -> unconnected-(U1-PA15-Pad38)
Routing:
- net GND: track 144.0 -> 131.5 mm, vias 5 -> 6
- net /SWDIO: track 26.4 -> 33.1 mm
- net /BOOT: track 22.6 -> 26.1 mm
- net +3.3V: track 70.9 -> 72.1 mm
- net /SCL: track 32.5 -> 33.4 mm
- net Net-(SW2-B): track 4.54 -> 3.74 mm
- net /SDA: track 28.8 -> 29.5 mm
