File: pcb/pcb.kicad_sch (KiCad schematic)
At the start: 20 parts, among them U1 STM32F103C8T6

Commit message: Change kicad version to 9.0.7
Parts:
- removed C? (x2): C, symbol Device:C
- removed C? (x5): 100n, symbol Device:C
- removed C? (x2): 33p, symbol Device:C
- removed C?: 10u, symbol Device:C
- removed D?: RED LED, symbol Device:LED
- removed J?: Conn_01x05_Pin, symbol Connector:Conn_01x05_Pin
- removed R? (x2): 10k, symbol Device:R
- removed SW? (x2): SW_SPDT, symbol Switch:SW_SPDT
- removed U?: AMS1117-3.3, Package_TO_SOT_SMD:SOT-223-3_TabPin2, symbol Regulator_Linear:AMS1117-3.3
- removed Y?: 8MHz, symbol Device:Crystal
- added C2, C? (x2): 10u, symbol Device:C
- added C3, C4, C5, C6: 100n, symbol Device:C
- added C? (x2): 33p, symbol Device:C
- added C?: C, symbol Device:C
- added J?: Conn_01x05_Pin, symbol Connector:Conn_01x05_Pin
- added R?: 10k, symbol Device:R
- added SW? (x2): SW_SPDT, symbol Switch:SW_SPDT
- added U?: AMS1117-3.3, Package_TO_SOT_SMD:SOT-223-3_TabPin2, symbol Regulator_Linear:AMS1117-3.3
- added Y?: 8MHz, symbol Device:Crystal
Connections:
- net +3.3V: now also C2.1, C3.1, C4.1, C5.1, C6.1, SW?.1 (A), SW?.2 (B)
- net BOOT: now also R?.2
- net GND: now also C2.2, C3.2, C4.2, C5.2, C6.2, C?.1, C?.1, C?.1, C?.2, C?.2, J?.5 (Pin_5), SW?.3 (C), U?.1 (GND)
- net HSE_IN: now also C?.2, Y?.2
- net HSE_OUT: now also C?.2, Y?.1
- net SWDCLK: now also J?.4 (Pin_4)
- net SWDIO: now also J?.3 (Pin_3)
- net NRST: no longer names the net of U1.7 (NRST)
- net NRST: now also C?.2
- new net: C?.1, SW?.1 (A), U?.2 (VO)
- new net: R?.1, SW?.2 (B)
- new net 3.3V_IN: J?.2 (Pin_2), SW?.3 (C)
- new net 5V_IN: C?.1, J?.1 (Pin_1), U?.3 (VI)

Commit message: Almost done with schematics
Parts:
- added C13, C7: 100n, symbol Device:C
- added D1, D2, D3, D4, D5, D6, D7, D8, D9: LED, symbol Device:LED
- added J1: Conn_01x03_Pin, symbol Connector:Conn_01x03_Pin
- added J2, J3, J6, J7: Conn_01x02_Pin, symbol Connector:Conn_01x02_Pin
- added J4: SPI2, symbol Connector:Conn_01x06_Pin
- added J8: I2C2, symbol Connector:Conn_01x04_Pin
- added J9: USART1, symbol Connector:Conn_01x04_Pin
- added R10, R11, R12, R2, R5, R6, R7, R8, R9: 1.5K, symbol Device:R
- added R3, R4: R, symbol Device:R
- added SW1: SW_Push, symbol Switch:SW_Push
- C11: renamed from C?; value C -> 100n
- J5: renamed from J?; value Conn_01x05_Pin -> SWD
- gave numbers to parts that had none: 9
Connections:
- net +3.3V: now also J2.1 (Pin_1), J3.1 (Pin_1), J4.1 (Pin_1), J8.1 (Pin_1), J9.1 (Pin_1), R2.2, R3.1, R4.1
- net 5V_IN: now also C7.1, J6.1 (Pin_1), J7.1 (Pin_1)
- net GND: now also C13.2, C7.2, D1.1 (K), J2.2 (Pin_2), J3.2 (Pin_2), J4.6 (Pin_6), J6.2 (Pin_2), J7.2 (Pin_2), J8.4 (Pin_4), J9.4 (Pin_4), R10.2, R11.2, R12.2, R5.2, R6.2, R7.2, R8.2, R9.2, SW1.1
- net at C12.1, SW3.1 (A), U2.2 (VO): now also C13.1
- net LED0: now reaches U1.10 (PA0)
- net LED0: now also D2.2 (A)
- net LED1: now reaches U1.11 (PA1)
- net LED1: now also D3.2 (A)
- net LED2: now reaches U1.12 (PA2)
- net LED2: now also D4.2 (A)
- net LED3: now reaches U1.13 (PA3)
- net LED3: now also D5.2 (A)
- net LED4: now reaches U1.14 (PA4)
- net LED4: now also D6.2 (A)
- net LED5: now reaches U1.15 (PA5)
- net LED5: now also D7.2 (A)
- net LED6: now reaches U1.16 (PA6)
- net LED6: now also D8.2 (A)
- net LED7: now reaches U1.17 (PA7)
- net LED7: now also D9.2 (A)
- net PC13: now reaches U1.2 (PC13)
- net PC13: now also J1.1 (Pin_1)
- net SCL: now reaches U1.21 (PB10)
- net SCL: now also J8.2 (Pin_2), R3.2
- net SDA: now reaches U1.22 (PB11)
- net SDA: now also J8.3 (Pin_3), R4.2
- net CS: now reaches U1.25 (PB12)
- net CS: now also J4.5 (Pin_5)
- net CLK: now reaches U1.26 (PB13)
- net CLK: now also J4.4 (Pin_4)
- net MISO: now reaches U1.27 (PB14)
- net MISO: now also J4.2 (Pin_2)
- net MOSI: now reaches U1.28 (PB15)
- net MOSI: now also J4.3 (Pin_3)
- net PC14: now reaches U1.3 (PC14)
- net PC14: now also J1.2 (Pin_2)
- net PC15: now reaches U1.4 (PC15)
- net PC15: now also J1.3 (Pin_3)
- net TX: now reaches U1.42 (PB6)
- net TX: now also J9.3 (Pin_3)
- net RX: now reaches U1.43 (PB7)
- net RX: now also J9.2 (Pin_2)
- net NRST: now reaches C11.2, U1.7 (NRST)
- net NRST: now also SW1.2
- new net: D6.1 (K), R9.1
- new net: D4.1 (K), R7.1
- new net: D5.1 (K), R8.1
- new net: D3.1 (K), R6.1
- new net: D2.1 (K), R5.1
- new net: D7.1 (K), R10.1
- new net: D8.1 (K), R11.1
- new net: D9.1 (K), R12.1
- new net: D1.2 (A), R2.1
- no-connect marks 0 -> 14
Other:
- title: (none) -> My Board
- moved on the sheet: C1, C10, C11, C12, C2, C3, C4, C5, C6, C8, C9, J5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

Commit message: Assigned footprints
Parts:
- C1, C10, C11, C12, C13, C2, C3, C4, C5, C6, C7, C8, C9: footprint (none) -> Capacitor_SMD:C_1206_3216Metric_Pad1.33x1.80mm_HandSolder
- D1, D2, D3, D4, D5, D6, D7, D8, D9: footprint (none) -> LED_SMD:LED_1206_3216Metric_Pad1.42x1.75mm_HandSolder
- J1: value Conn_01x03_Pin -> GPIO; footprint (none) -> Connector_PinHeader_2.54mm:PinHeader_1x03_P2.54mm_Vertical
- J2, J3: value Conn_01x02_Pin -> 3.3V Power; footprint (none) -> Connector_PinHeader_2.54mm:PinHeader_1x02_P2.54mm_Vertical
- J4: footprint (none) -> Connector_PinSocket_2.54mm:PinSocket_1x06_P2.54mm_Vertical
- J5: footprint (none) -> Connector_PinSocket_2.54mm:PinSocket_1x05_P2.54mm_Vertical
- J6, J7: value Conn_01x02_Pin -> 5V Power; footprint (none) -> Connector_PinHeader_2.54mm:PinHeader_1x02_P2.54mm_Vertical
- J8, J9: footprint (none) -> Connector_PinSocket_2.54mm:PinSocket_1x04_P2.54mm_Vertical
- R1, R10, R11, R12, R2, R3, R4, R5, R6, R7, R8, R9: footprint (none) -> Resistor_SMD:R_1206_3216Metric_Pad1.30x1.75mm_HandSolder
- SW1: footprint (none) -> Button_Switch_SMD:SW_SPST_PTS647_Sx38
- SW2, SW3: footprint (none) -> Button_Switch_SMD:SW_SPDT_PCM12
- Y1: footprint (none) -> Crystal:Crystal_SMD_HC49-SD

Commit message: PCB mid-way
Parts:
- J4: footprint Connector_PinSocket_2.54mm:PinSocket_1x06_P2.54mm_Vertical -> Connector_PinHeader_2.54mm:PinHeader_1x06_P2.54mm_Vertical
- J5: footprint Connector_PinSocket_2.54mm:PinSocket_1x05_P2.54mm_Vertical -> Connector_PinHeader_2.54mm:PinHeader_1x05_P2.54mm_Vertical
- J8, J9: footprint Connector_PinSocket_2.54mm:PinSocket_1x04_P2.54mm_Vertical -> Connector_PinHeader_2.54mm:PinHeader_1x04_P2.54mm_Vertical
Changed lines of the file:
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@@
 			)
 		)
-		(property "Footprint" "Connector_PinSocket_2.54mm:PinSocket_1x06_P2.54mm_Vertical"
+		(property "Footprint" "Connector_PinHeader_2.54mm:PinHeader_1x06_P2.54mm_Vertical"
 			(at 176.53 142.24 0)
 			(effects
@@
 			)
 		)
-		(property "Footprint" "Connector_PinSocket_2.54mm:PinSocket_1x04_P2.54mm_Vertical"
+		(property "Footprint" "Connector_PinHeader_2.54mm:PinHeader_1x04_P2.54mm_Vertical"
 			(at 208.28 118.11 0)
 			(effects
@@
 			)
 		)
-		(property "Footprint" "Connector_PinSocket_2.54mm:PinSocket_1x05_P2.54mm_Vertical"
+		(property "Footprint" "Connector_PinHeader_2.54mm:PinHeader_1x05_P2.54mm_Vertical"
 			(at 176.53 119.38 0)
 			(effects
@@
 			)
 		)
-		(property "Footprint" "Connector_PinSocket_2.54mm:PinSocket_1x04_P2.54mm_Vertical"
+		(property "Footprint" "Connector_PinHeader_2.54mm:PinHeader_1x04_P2.54mm_Vertical"
 			(at 207.01 140.97 0)
 			(effects

Commit message: PCB almost done, proctored by Parul
Connections:
- net CLK: now also J4.3 (Pin_3); no longer J4.4 (Pin_4)
- net CS: now also J4.2 (Pin_2); no longer J4.5 (Pin_5)
- net MISO: now also J4.4 (Pin_4); no longer J4.2 (Pin_2)
- net MOSI: now also J4.5 (Pin_5); no longer J4.3 (Pin_3)
Changed lines of the file:
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@@
-	(wire
-		(pts
-			(xy 181.61 139.7) (xy 187.96 139.7)
-		)
-		(stroke
-			(width 0)
-			(type default)
-		)
-	)
 	(wire
 		(pts
@@
 	(wire
 		(pts
+			(xy 181.61 147.32) (xy 186.69 147.32)
+		)
+		(stroke
+			(width 0)
+			(type default)
+		)
+	)
+	(wire
+		(pts
 			(xy 217.17 120.65) (xy 213.36 120.65)
 		)
@@
 	(wire
 		(pts
+			(xy 181.61 144.78) (xy 186.69 144.78)
+		)
+		(stroke
+			(width 0)
+			(type default)
+		)
+	)
+	(wire
+		(pts
 			(xy 123.19 77.47) (xy 120.65 77.47)
 		)
@@
 	(wire
 		(pts
+			(xy 181.61 139.7) (xy 186.69 139.7)
+		)
+		(stroke
+			(width 0)
+			(type default)
+		)
+	)
+	(wire
+		(pts
 			(xy 22.86 38.1) (xy 27.94 38.1)
 		)
@@
 	(wire
 		(pts
-			(xy 181.61 144.78) (xy 187.96 144.78)
-		)
-		(stroke
-			(width 0)
-			(type default)
-		)
-	)
-	(wire
-		(pts
 			(xy 181.61 137.16) (xy 182.88 137.16)
 		)
@@
 	(wire
 		(pts
+			(xy 181.61 142.24) (xy 186.69 142.24)
+		)
+		(stroke
+			(width 0)
+			(type default)
+		)
+	)
+	(wire
+		(pts
 			(xy 273.05 80.01) (xy 273.05 88.9)
 		)
@@
 	(wire
 		(pts
-			(xy 181.61 147.32) (xy 187.96 147.32)
-		)
-		(stroke
-			(width 0)
-			(type default)
-		)
-	)
-	(wire
-		(pts
 			(xy 118.11 161.29) (xy 120.65 161.29)
 		)
@@
 		(pts
 			(xy 22.86 39.37) (xy 22.86 38.1)
-		)
-		(stroke
-			(width 0)
-			(type default)
-		)
-	)
-	(wire
-		(pts
-			(xy 181.61 142.24) (xy 187.96 142.24)
 		)
 		(stroke
@@
 	)
 	(label "CS"
-		(at 187.96 147.32 180)
+		(at 186.69 139.7 180)
 		(effects
 			(font
@@
 	)
 	(label "CLK"
-		(at 187.96 144.78 180)
+		(at 186.69 142.24 180)
 		(effects
 			(font
@@
 	)
 	(label "MISO"
-		(at 187.96 139.7 180)
+		(at 186.69 144.78 180)
 		(effects
 			(font
@@
 	)
 	(label "MOSI"
-		(at 187.96 142.24 180)
-		(effects
-			(font
+		(at 186.69 147.32 180)
+		(effects
+			(font

Commit message: Completed routing with some silkscreen
Connections:
- net SCL: now also J8.3 (Pin_3), R4.2; no longer J8.2 (Pin_2), R3.2
- net SDA: now also J8.2 (Pin_2), R3.2; no longer J8.3 (Pin_3), R4.2
Changed lines of the file:
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@@
+	(wire
+		(pts
+			(xy 212.09 140.97) (xy 218.44 140.97)
+		)
+		(stroke
+			(width 0)
+			(type default)
+		)
+	)
 	(wire
 		(pts
@@
 	(wire
 		(pts
-			(xy 218.44 140.97) (xy 212.09 140.97)
-		)
-		(stroke
-			(width 0)
-			(type default)
-		)
-	)
-	(wire
-		(pts
 			(xy 91.44 100.33) (xy 100.33 100.33)
 		)
@@
 	(wire
 		(pts
-			(xy 218.44 143.51) (xy 212.09 143.51)
-		)
-		(stroke
-			(width 0)
-			(type default)
-		)
-	)
-	(wire
-		(pts
 			(xy 226.06 140.97) (xy 227.33 140.97)
 		)
@@
 		(pts
 			(xy 120.65 77.47) (xy 120.65 80.01)
+		)
+		(stroke
+			(width 0)
+			(type default)
+		)
+	)
+	(wire
+		(pts
+			(xy 212.09 143.51) (xy 218.44 143.51)
 		)
 		(stroke
@@
 	)
 	(label "SCL"
-		(at 215.9 140.97 180)
+		(at 215.9 143.51 180)
 		(effects
 			(font
@@
 	)
 	(label "SDA"
-		(at 215.9 143.51 180)
-		(effects
-			(font
+		(at 215.9 140.97 180)
+		(effects
+			(font

Commit message: Finished PCB
Connections:
- net SWDCLK: now also U1.37 (PA14); no longer U1.38 (PA15)
- net SWDIO: now also U1.34 (PA13); no longer U1.37 (PA14)
Changed lines of the file:
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@@
+	)
+	(no_connect
+		(at 135.89 125.73)
 	)
 	(no_connect
@@
 	)
 	(no_connect
-		(at 135.89 120.65)
-	)
-	(no_connect
 		(at 135.89 110.49)
 	)
@@
 	(wire
 		(pts
+			(xy 135.89 123.19) (xy 144.78 123.19)
+		)
+		(stroke
+			(width 0)
+			(type default)
+		)
+	)
+	(wire
+		(pts
 			(xy 241.3 80.01) (xy 248.92 80.01)
 		)
@@
 	(wire
 		(pts
+			(xy 135.89 120.65) (xy 144.78 120.65)
+		)
+		(stroke
+			(width 0)
+			(type default)
+		)
+	)
+	(wire
+		(pts
 			(xy 95.25 140.97) (xy 100.33 140.97)
 		)
@@
 	(wire
 		(pts
-			(xy 135.89 125.73) (xy 144.78 125.73)
-		)
-		(stroke
-			(width 0)
-			(type default)
-		)
-	)
-	(wire
-		(pts
 			(xy 266.7 63.5) (xy 273.05 63.5)
 		)
@@
 		(pts
 			(xy 241.3 63.5) (xy 248.92 63.5)
-		)
-		(stroke
-			(width 0)
-			(type default)
-		)
-	)
-	(wire
-		(pts
-			(xy 135.89 123.19) (xy 144.78 123.19)
 		)
 		(stroke
@@
 	)
 	(label "SWDCLK"
-		(at 144.78 125.73 180)
+		(at 144.78 123.19 180)
 		(effects
 			(font
@@
 	)
 	(label "SWDIO"
-		(at 144.78 123.19 180)
-		(effects
-			(font
+		(at 144.78 120.65 180)
+		(effects
+			(font

Commit message: Cleaned up the schematics
Other:
- note added: "3.3v OUT"
- note added: "5v OUT"
- note added: "BOOT"
- note added: "GPIO"
- note added: "HSE"
- note added: "I2C"
- note added: "LED SERIES"
- note added: "NRST"
- note added: "POWER CIRCUIT"
- note added: "SPI"
- note added: "SWD"
- note added: "UART"
- moved on the sheet: C1, C10, C11, C12, C13, C2, C3, C4, C5, C6, C7, C8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
